File: PaperPlane/PaperPlane.kicad_pcb (KiCad board)
At the start: 2 copper layers, 6 parts

Commit message: HalfFinish
Parts:
- added BATT1: Conn_01x02_Male, Connector_JST:JST_PH_B2B-PH-K_1x02_P2.00mm_Vertical, F.Cu at (252.2, 124.8)
- added CMotor1: 0.1uF, Capacitor_SMD:C_0603_1608Metric, F.Cu at (272.6, 108.6)
- added CMotor2: 0.1uF, Capacitor_SMD:C_0603_1608Metric, F.Cu at (272.6, 113.6)
- added CRST1: 0.1uF, Capacitor_SMD:C_0603_1608Metric, F.Cu at (264.7, 120.6)
- added LED1: LED, LED_SMD:LED_0603_1608Metric, F.Cu at (278.2, 126.5)
- added MOTOR1: Conn_01x02_Male, Connector_JST:JST_PH_B2B-PH-K_1x02_P2.00mm_Vertical, F.Cu at (265.6, 110.0)
- added ON1: LED, LED_SMD:LED_0603_1608Metric, F.Cu at (282.3, 126.5)
- added R-RST1: 10k, Resistor_SMD:R_0603_1608Metric, F.Cu at (258.7, 129.8)
- added RBOOT1: 10k, Resistor_SMD:R_0603_1608Metric, F.Cu at (272.1, 116.1)
- added RLED1: 1k, Resistor_SMD:R_0603_1608Metric, F.Cu at (265.6, 123.1)
- added RON1: 1k, Resistor_SMD:R_0603_1608Metric, F.Cu at (268.7, 120.6)
- added RRX1: 22R, Resistor_SMD:R_0603_1608Metric, F.Cu at (272.6, 111.1)
- added RTX1: 22R, Resistor_SMD:R_0603_1608Metric, F.Cu at (258.7, 132.3)
- added STM32G311: STM32G031K8T6, Package_QFP:LQFP-32_7x7mm_P0.8mm, F.Cu at (208.8, 125.0)
- added SW-RST1: SW_Push, Switches:TACTILE_SWITCH_SMD_6.0X3.5MM, F.Cu at (267.5, 105.0)
- added Servo1: Conn_01x03_Male, Connector_Hirose:Hirose_DF13-03P-1.25DSA_1x03_P1.25mm_Vertical, F.Cu at (265.1, 117.1)
- added Servo2: Conn_01x03_Male, Connector_Hirose:Hirose_DF13-03P-1.25DSA_1x03_P1.25mm_Vertical, F.Cu at (251.8, 131.8)
- added Servo3: Conn_01x03_Male, Connector_PinHeader_2.54mm:PinHeader_1x03_P2.54mm_Horizontal, F.Cu at (251.6, 114.7)
- added Servo4: Conn_01x03_Male, Connector_PinHeader_2.54mm:PinHeader_1x03_P2.54mm_Horizontal, F.Cu at (251.6, 105.0)
- added U1: MPU-6050, Sensor_Motion:InvenSense_QFN-24_4x4mm_P0.5mm, F.Cu at (260.4, 125.2)
- added U2: ESP32-WROOM-32, RF_Module:ESP32-WROOM-32, F.Cu at (234.5, 124.2)
- added U3: DRV8837C, Package_SON:WSON-8-1EP_2x2mm_P0.5mm_EP0.9x1.6mm, F.Cu at (274.4, 104.4)
- added UART1: Conn_01x04_Female, Connector_PinSocket_2.54mm:PinSocket_1x04_P2.54mm_Vertical, F.Cu at (273.9, 127.5)
- added Y1: Crystal_GND24, Crystal:Crystal_SMD_3225-4Pin_3.2x2.5mm, F.Cu at (217.1, 121.5)
